Commit message: new updates

File: ros2_ws/src/basic_gazebo_rviz_demo/models/model.urdf (robot description, URDF)
Before this commit: robot simple_robot, 3 links, 2 joints
Links:
- added link base_footprint
- added link caster_wheel; visual sphere radius=0.025
Joints:
- added joint base_caster_joint: type fixed, parent base_link, child caster_wheel, origin xyz=-0.15 0 -0.025 rpy=0 0 0
- added joint base_joint: type fixed, parent base_footprint, child base_link, origin xyz=0 0 -0.5 rpy=0 0 0
